Commit message: 5월 17일 연구

File: local_assets/roarm_m3/urdf/roarm_m3.urdf (robot description, URDF)
Before this commit: robot roarm_m3, 9 links, 8 joints
Links:
- link gripper_link: geometry collision mesh filename=meshes/gripper_link_collision_g2a.stl scale=0.001 0.001 0.001; visual mesh filename=meshes/gripper_link.stl scale=0.001 0.001 0.001
