Commit message: 그랩 v1 체결구 검증 BLOCKED(D475) → g18_nut_trap 3점 체결·포켓 너트로 해소(D476) + URDF/USD 재생성
- p38 체결구 프로브 신설: 간극 4.05 − 크랭크판 3.0 = 잔여 1.03 에 브래킷 너트·크랭크 머리가 같은 자리 → BLOCKED
- 설계 수정: 브래킷 Z 102.9 쌍(바깥 볼트·안쪽 너트) + 팁 구멍(레일 슬롯 너트), 크랭크판 포켓 너트, 판 폭 link5 플랜지 안쪽, BOM 7종, 자중 58.53 g
- p37 정정: G3 실기하 래스터 대조(옛 판 구멍이 중앙선에 있던 거짓 PASS), G6 플랜지 검사(옛 판 link5 관통), AABB 하한 정확 재측정
- 설계 19/20 · p37 G2_ATTACH_OK · p38 G2_DRIVE_EXTRACTION_OK
- URDF/USD 재생성: convert_mimic_joints_to_normal_joints=False (True 는 PhysX mimic 생성 — 플래그 반전, D477)

Co-Authored-By: Claude Fable 5.1 <noreply@anthropic.com>
Claude-Session: https://claude.ai/code/session_0155ufus1ZSatosQjH3ETj4f

File: local_assets/roarm_m3/urdf/roarm_m3_with_grab.urdf (robot description, URDF)
Before this commit: robot roarm_m3, 12 links, 11 joints
Links:
- link grab_base: mass 0.0152484 -> 0.0129942; geometry collision mesh filename=meshes/collision/bracket_bolt_plate_0.stl scale=0.001 0.001 0.001; collision mesh filename=meshes/collision/bracket_bolt_plate_1.stl scale=0.001 0.001 0.001
