Commit message: 정밀 collision (조각별 볼록 STL) + Isaac 렌더/변환 스크립트
■ 정밀 collision (사용자 요청)
export_grab_urdf.py: 링크 collision 을 **볼록 조각별 STL**로 (visual=병합 _ALL 1개 · collision=조각별).
각 조각이 all_pieces_convex 통과 = 볼록 → convexHull=자기 자신 → union=정확한 오목 공동.
convex_decomposition(VHACD 근사)보다 정확. 조각 수: bracket 110 · shell_L 120 · shell_R 120 = 350.
compose_roarm_grab_urdf.py: collision 조각을 로봇 meshes/collision/ 로 복사.
sim_urdf_to_usd.py: --collider {convex_hull,convex_decomposition} 인자화 (조각별이면 convex_hull=정확).

■ 검증 (pxr)
USD 재임포트(convex_hull) → 그랩 링크별 collision 메시 350개(110/120/120) · 근사 convexHull 확인.
링크 6/6·조인트 11 온전. D446(단일 hull 이 스쿱 공동 채움) 근본 회피.

■ Isaac 렌더 (sim_render_grab_usd.py)
합성 USD 를 Isaac Sim 5.1 RTX 헤드리스 렌더 → PNG. 스쿱 자세 + 그랩 개방, 중력 off 로 자세 유지.

collision STL(local_assets, 1.4MB) 커밋 = 자족적 로봇 자산. g17 중간 collision·isaac_render.png·USD 는 gitignore(regenerable).

Co-Authored-By: Claude Fable 5 <noreply@anthropic.com>
Claude-Session: https://claude.ai/code/session_01WwvdYNrTy7JkrrWK49bzVX

File: claudedocs/runtime_logs/grab_track/g17_yoke_alu/urdf/grab_v1.urdf (robot description, URDF)
Before this commit: robot grab_v1, 3 links, 2 joints
Links:
- link grab_base: geometry collision mesh filename=meshes/collision/bracket_bolt_plate_0.stl scale=0.001 0.001 0.001; collision mesh filename=meshes/collision/bracket_bolt_plate_1.stl scale=0.001 0.001 0.001
- link grab_shell_L: geometry collision mesh filename=meshes/collision/shell_L_bowl_00.stl scale=0.001 0.001 0.001; collision mesh filename=meshes/collision/shell_L_bowl_01.stl scale=0.001 0.001 0.001
- link grab_shell_R: geometry collision mesh filename=meshes/collision/shell_R_bowl_00.stl scale=0.001 0.001 0.001; collision mesh filename=meshes/collision/shell_R_bowl_01.stl scale=0.001 0.001 0.001

File: local_assets/roarm_m3/urdf/roarm_m3_with_grab.urdf (robot description, URDF)
Before this commit: robot roarm_m3, 12 links, 11 joints
Links:
- link grab_base: geometry collision mesh filename=meshes/collision/bracket_bolt_plate_0.stl scale=0.001 0.001 0.001; collision mesh filename=meshes/collision/bracket_bolt_plate_1.stl scale=0.001 0.001 0.001
- link grab_shell_L: geometry collision mesh filename=meshes/collision/shell_L_bowl_00.stl scale=0.001 0.001 0.001; collision mesh filename=meshes/collision/shell_L_bowl_01.stl scale=0.001 0.001 0.001
- link grab_shell_R: geometry collision mesh filename=meshes/collision/shell_R_bowl_00.stl scale=0.001 0.001 0.001; collision mesh filename=meshes/collision/shell_R_bowl_01.stl scale=0.001 0.001 0.001
